Commit message: description: track_width 0.400 -> 0.190 measured drive-wheel spacing
Drive wheels sit inside the body shell; stored value was the body
width, which skewed kinematics and odometry.

File: src/helper_description/urdf/helper_robot.urdf.xacro (robot description, xacro)
@@ -3,5 +3,6 @@
   <xacro:property name="wheel_radius" value="0.065"/>
   <xacro:property name="wheel_width" value="0.03"/>
-  <xacro:property name="track_width" value="0.400"/>
+  <!-- Measured drive-wheel center spacing; wheels sit inside the body shell. -->
+  <xacro:property name="track_width" value="0.190"/>
   <xacro:property name="base_length" value="0.400"/>
   <xacro:property name="base_width" value="0.320"/>
